File: hardware/power/fets.kicad_sch (KiCad schematic)
At the start: 6 parts, among them Q201 ISC022N10NM6, Q202 ISC022N10NM6, Q203 ISC022N10NM6, Q204 ISC022N10NM6, Q205 ISC022N10NM6, Q206 ISC022N10NM6

Commit message: added connectors to add individual current paths, filled with ntcs, plotted pdf, updated screenshots
Other:
- company: openmc -> github.com/arminstr
Changed lines of the file:
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@@
 		(date "2025-09-12")
 		(rev "${REV}")
-		(company "openmc")
-		(comment 1 "Armin S.")
+		(company "github.com/arminstr")
 	)
 	(junction
